Commit message: updated ridgeback_description, will need to tune IMU depending on real config

File: src/ridgeback/ridgeback_description_lasa/urdf/accessories.urdf.xacro (robot description, xacro)
@@ -10,4 +10,5 @@
   -->
   <xacro:include filename="$(find ridgeback_description)/urdf/accessories/sick_lms1xx_mount.urdf.xacro" />
+  <xacro:include filename="$(find ridgeback_description)/urdf/accessories/sick_s300_mount.urdf.xacro" />
   <xacro:include filename="$(find ridgeback_description)/urdf/accessories/hokuyo_ust-10lx_mount.urdf.xacro" />
   <xacro:include filename="$(find ur_description)/urdf/inc/ur5_macro.xacro" />
@@ -15,25 +16,65 @@
   <xacro:if value="$(optenv RIDGEBACK_FRONT_HOKUYO_LASER 0)">
     <xacro:hokuyo_ust-10lx_mount prefix="front"
-                            topic="front/scan"
-                            location="1" />
+                                 topic="front/scan"
+                                 location="1" />
   </xacro:if>
   <!-- If enabled, generate the rear HOKUYO UST-10LX LASER payload. -->
   <xacro:if value="$(optenv RIDGEBACK_REAR_HOKUYO_LASER 0)">
     <xacro:hokuyo_ust-10lx_mount prefix="rear"
-                            topic="rear/scan"
-                            location="-1" />
+                                 topic="rear/scan"
+                                 location="-1" />
   </xacro:if>
   <!-- If enabled, generate the front SICK LMS111 LASER payload. -->
   <xacro:if value="$(optenv RIDGEBACK_FRONT_SICK_LASER 0)">
     <xacro:sick_lms1xx_mount prefix="front"
-                            topic="front/scan"
-                            location="1" />
+                             topic="front/scan"
+                             location="1" />
   </xacro:if>
   <!-- If enabled, generate the rear SICK LMS111 LASER payload. -->
   <xacro:if value="$(optenv RIDGEBACK_REAR_SICK_LASER 0)">
     <xacro:sick_lms1xx_mount prefix="rear"
-                            topic="rear/scan"
-                            location="-1" />
+                             topic="rear/scan"
+                             location="-1" />
   </xacro:if>
+  <!-- If enabled, generate the front SICK S300 LASER payload.
+       This uses the same mesh as the lms1xx since they are the footprint
+       and the simulation parameters can be variable. -->
+  <xacro:if value="$(optenv RIDGEBACK_FRONT_S300_LASER 0)">
+    <xacro:sick_s300_mount prefix="front"
+                             topic="front/scan"
+                             location="1" />
+  </xacro:if>
+  <!-- If enabled, generate the rear SICK S300 LASER payload. -->
+  <xacro:if value="$(optenv RIDGEBACK_REAR_S300_LASER 0)">
+    <xacro:sick_s300_mount prefix="rear"
+                             topic="rear/scan"
+                             location="-1" />
+  </xacro:if>
+  <!-- Legacy support for Microstrain IMU GX2 -->
+  <xacro:include filename="$(find ridgeback_description)/urdf/accessories/microstrain_imu.urdf.xacro" />
+  <xacro:if value="$(optenv RIDGEBACK_MICROSTRAIN_IMU 0)">
+    <xacro:microstrain_imu prefix="$(optenv RIDGEBACK_MICROSTRAIN_IMU_PREFIX upgraded)"
+                           mount_link="$(optenv RIDGEBACK_MICROSTRAIN_IMU_MOUNT mid)_mount" >
+      <origin xyz="$(optenv RIDGEBACK_MICROSTRAIN_IMU_OFFSET 0 0 0)"
+              rpy="$(optenv RIDGEBACK_MICROSTRAIN_IMU_RPY 0 0 0)" />
+    </xacro:microstrain_imu>
+  </xacro:if>
+  <!--
+    Support for current Microstrain IMU models, including GX3, GX5, GX25, etc. By default the Ridgeback comes equipped with an IMU linked to "imu_link". These extra optional microstrain IMU's will be added to another frame, by default, "microstrain_link".
+  -->
+  <xacro:if value="$(optenv RIDGEBACK_IMU_MICROSTRAIN 0)">
+    <xacro:property name="frame"  value="$(optenv RIDGEBACK_IMU_MICROSTRAIN_LINK microstrain_link)"/>
+    <xacro:property name="parent" value="$(optenv RIDGEBACK_IMU_MICROSTRAIN_PARENT base_link)"/>
+    <xacro:property name="xyz"    value="$(optenv RIDGEBACK_IMU_MICROSTRAIN_OFFSET -0.139 0.096 0.100)"/>
+    <xacro:property name="rpy"    value="$(optenv RIDGEBACK_IMU_MICROSTRAIN_RPY ${PI} 0 -${PI/2})"/>
+    <link name="${frame}" />
+    <joint name="${frame}_joint" type="fixed">
+      <parent link="${parent}" />
+      <child link="${frame}" />
+      <origin xyz="${xyz}" rpy="${rpy}" />
+    </joint>
+  </xacro:if>
+  <!-- Adding LASA specific accessories starting here -->
+  <!-- Spawn arch from dae file-->
   <link name="arch_link">
 		<visual>
@@ -49,9 +90,9 @@
    </link>
   <joint name="arch_joint" type="fixed">
-	  <origin xyz="-0.38 0 0.278" rpy="0 0 1.5" />
+	  <origin xyz="-0.38 0 0.278" rpy="0 0 1.5707" />
 	  <parent link="top_link" />
 	  <child link="arch_link" />
   </joint>
-<!-- Spawn arm -->
+  <!-- Spawn arm -->
   <xacro:ur5_robot prefix="ur5_arm_"/>
   <!-- Join arm -->
@@ -61,5 +102,5 @@
 	<origin xyz="0.22 0.0 0.0" rpy="0.0 0.0 -1.5708" />
   </joint>
-  <!-- Sensor Mount and other custom parts -->
+  <!-- Spawn F/T sensor -->
   <link name="FT300_link">
 		<visual>

File: src/ridgeback/ridgeback_description_lasa/urdf/accessories/hokuyo_ust-10lx_mount.urdf.xacro (robot description, xacro)
@@ -31,5 +31,5 @@
     </link>
     <gazebo reference="${prefix}_laser">
-      <turnGravityOff>true</turnGravityOff>
+      <turnGravityOff>false</turnGravityOff>
       <sensor type="ray" name="${prefix}_laser">
         <pose>0 0 0 0 0 0</pose>
@@ -62,4 +62,5 @@
         </plugin>
       </sensor>
+      <material>Gazebo/DarkGrey</material>
     </gazebo>
   </xacro:macro>

File: src/ridgeback/ridgeback_description_lasa/urdf/ridgeback.urdf.xacro (robot description, xacro)
@@ -8,13 +8,19 @@
   <xacro:property name="chassis_height" value="0.216" />
   <xacro:property name="deck_height" value="0.280" />
+  <xacro:property name="deck_thickness" value="0.005" />
+  <xacro:property name="riser_height" value="$(optenv RIDGEBACK_RISER_HEIGHT 0.055)" />
   <xacro:property name="axle_offset" value="0.0500" />
   <xacro:property name="rocker_offset" value="0.319" />
   <xacro:property name="rocker_width" value="0.472" />
+  <xacro:property name="imu_offset_x" value="0.2085" />
+  <xacro:property name="imu_offset_y" value="-0.2902" />
+  <xacro:property name="imu_offset_z" value="0.1681" />
   <xacro:property name="dummy_inertia" value="1e-09"/>
   <material name="dark_grey"><color rgba="0.2 0.2 0.2 1.0" /></material>
   <material name="light_grey"><color rgba="0.4 0.4 0.4 1.0" /></material>
+  <material name="red"><color rgba="0.8 0.0 0.0 1.0" /></material>
+  <material name="white"><color rgba="0.9 0.9 0.9 1.0" /></material>
   <material name="yellow"><color rgba="0.8 0.8 0.0 1.0" /></material>
   <material name="black"><color rgba="0.15 0.15 0.15 1.0" /></material>
-  <!-- added in accessories <xacro:include filename="$(find ur_description)/urdf/ur5.urdf.xacro" />-->
   <xacro:macro name="wheel" params="prefix side *joint_pose">
     <link name="${prefix}_${side}_wheel_link">
@@ -34,9 +40,9 @@
       <inertial>
         <origin xyz="0 0 0" rpy="0 0 0"/>
-        <mass value="0.477"/>
+        <mass value="2.3"/>
         <inertia
-          ixx="0.0013" ixy="0" ixz="0"
-          iyy="0.0024" iyz="0"
-          izz="0.0013"/>
+          ixx="3.3212e-3" ixy="0" ixz="0"
+          iyy="6.6424e-3" iyz="0"
+          izz="3.3212e-3"/>
       </inertial>
     </link>
@@ -50,5 +56,5 @@
       <type>transmission_interface/SimpleTransmission</type>
       <joint name="${prefix}_${side}_wheel">
-        <hardwareInterface>VelocityJointInterface</hardwareInterface>
+        <hardwareInterface>hardware_interface/VelocityJointInterface</hardwareInterface>
       </joint>
       <actuator name="${prefix}_${side}_actuator">
@@ -67,10 +73,10 @@
       </visual>
       <inertial>
-        <origin xyz="0 0 0" rpy="0 0 0"/>
-        <mass value="3"/>
+        <origin xyz="0 0 0" rpy="${PI/2} 0 ${PI/2}"/>
+        <mass value="10.267"/>
         <inertia
-          ixx="0.001" ixy="0" ixz="0"
-          iyy="0.001" iyz="0"
-          izz="0.001"/>
+          ixx="0.0288" ixy="2.20484e-6" ixz="-1.3145e-5"
+          iyy="0.4324" iyz="1.8944e-3"
+          izz="0.4130"/>
       </inertial>
     </link>
@@ -103,5 +109,5 @@
   <link name="chassis_link">
     <visual>
-      <origin xyz="0 0 0" rpy=" ${PI/2} 0 ${PI/2}" />
+      <origin xyz="0 0 0" rpy="0 0 0" />
       <geometry>
         <mesh filename="package://ridgeback_description/meshes/body.stl"/>
@@ -110,18 +116,66 @@
     </visual>
     <collision>
-      <origin xyz="0 0 ${chassis_height/2}"/>
-      <geometry>
-        <box size="${chassis_length} ${chassis_width} ${chassis_height}"/>
+      <origin xyz="0 0 0"/>
+      <geometry>
+        <mesh filename="package://ridgeback_description/meshes/body-collision.stl"/>
       </geometry>
     </collision>
     <inertial>
-      <origin xyz="0.012 0.002 0.067" rpy="0 0 0"/>
-      <mass value="50"/>
+      <origin xyz="0.012 0.002 0.067" rpy="${PI/2} 0 ${PI/2}"/>
+      <mass value="165.304"/>
       <inertia
-        ixx="1.3136" ixy="0.0" ixz="0.0"
-        iyy="1.3922" iyz="0.0"
-        izz="2.0"/>
+        ixx="4.4744" ixy="0.03098" ixz="0.003647"
+        iyy="7.1624" iyz="0.1228"
+        izz="4.6155"/>
     </inertial>
   </link>
+  <link name="riser_link">
+    <visual>
+      <origin xyz="0 0 ${riser_height/2}" rpy="0 0 ${pi/4}" />
+      <geometry>
+        <box size="0.493 0.493 ${riser_height}" />
+      </geometry>
+      <material name="light_grey" />
+    </visual>
+    <collision>
+      <origin xyz="0 0 ${riser_height/2}" rpy="0 0 ${pi/4}" />
+      <geometry>
+        <box size="0.493 0.493 ${riser_height}" />
+      </geometry>
+    </collision>
+  </link>
+  <joint name="riser_link_joint" type="fixed">
+    <origin xyz="0 0 ${0.225 - deck_thickness}" rpy="0 0 0" />
+    <parent link="chassis_link" />
+    <child link="riser_link" />
+  </joint>
+  <joint name="right_side_cover_link_joint" type="fixed">
+    <origin xyz="0 0 0" rpy="0 0 0" />
+    <parent link="chassis_link"/>
+    <child link="right_side_cover_link" />
+  </joint>
+  <joint name="left_side_cover_link_joint" type="fixed">
+    <origin xyz="0 0 0" rpy="0 0 0" />
+    <parent link="chassis_link"/>
+    <child link="left_side_cover_link" />
+  </joint>
+  <link name="left_side_cover_link">
+    <visual>
+      <origin xyz="0 0 0" rpy="0 0 ${PI}" />
+      <geometry>
+        <mesh filename="package://ridgeback_description/meshes/side-cover.stl"/>
+      </geometry>
+      <material name="yellow" />
+    </visual>
+  </link>
+  <link name="right_side_cover_link">
+    <visual>
+      <origin xyz="0 0 0" rpy="0 0 0" />
+      <geometry>
+        <mesh filename="package://ridgeback_description/meshes/side-cover.stl"/>
+      </geometry>
+      <material name="yellow" />
+    </visual>
+  </link>
   <joint name="front_cover_link_joint" type="fixed">
     <origin xyz="0 0 0" rpy="0 0 0" />
@@ -131,5 +185,5 @@
   <link name="front_cover_link">
     <visual>
-      <origin xyz="0 0 0" rpy=" ${PI/2} 0 ${-PI/2}"  />
+      <origin xyz="0 0 0" rpy="0 0 0" />
       <geometry>
         <mesh filename="package://ridgeback_description/meshes/end-cover.stl" />
@@ -145,5 +199,5 @@
   <link name="rear_cover_link">
     <visual>
-      <origin xyz="0 0 0" rpy=" ${PI/2} 0 ${PI/2}"  />
+      <origin xyz="0 0 0" rpy="0 0 ${PI}" />
       <geometry>
         <mesh filename="package://ridgeback_description/meshes/end-cover.stl" />
@@ -152,12 +206,40 @@
     </visual>
   </link>
+  <joint name="front_lights_link_joint" type="fixed">
+    <origin xyz="0 0 0" rpy="0 0 0" />
+    <parent link="chassis_link"/>
+    <child link="front_lights_link" />
+  </joint>
+  <joint name="rear_lights_link_joint" type="fixed">
+    <origin xyz="0 0 0" rpy="0 0 0" />
+    <parent link="chassis_link"/>
+    <child link="rear_lights_link" />
+  </joint>
+  <link name="front_lights_link">
+    <visual>
+      <origin xyz="0 0 0" rpy="0 0 0" />
+      <geometry>
+        <mesh filename="package://ridgeback_description/meshes/lights.stl" />
+      </geometry>
+      <material name="white" />
+    </visual>
+  </link>
+  <link name="rear_lights_link">
+    <visual>
+      <origin xyz="0 0 0" rpy="0 0 ${PI}" />
+      <geometry>
+        <mesh filename="package://ridgeback_description/meshes/lights.stl" />
+      </geometry>
+      <material name="black" />
+    </visual>
+  </link>
   <joint name="top_link_joint" type="fixed">
-    <origin xyz="0 0 0" rpy="0 0 0" />
-    <parent link="chassis_link"/>
+    <origin xyz="0 0 ${riser_height-deck_height+deck_thickness}" rpy="0 0 0" />
+    <parent link="riser_link"/>
     <child link="top_link" />
   </joint>
   <link name="top_link">
     <visual>
-      <origin xyz="${-chassis_length/2} ${-chassis_width/2} 0" rpy=" ${PI/2} 0 ${PI/2}" />
+      <origin xyz="0 0 0" rpy="0 0 0" />
       <geometry>
         <mesh filename="package://ridgeback_description/meshes/top.stl" />
@@ -165,4 +247,10 @@
       <material name="black" />
     </visual>
+    <collision>
+      <origin xyz="0 0 0" rpy="0 0 0" />
+      <geometry>
+        <mesh filename="package://ridgeback_description/meshes/top.stl"/>
+      </geometry>
+    </collision>
   </link>
   <joint name="axle_joint" type="fixed">
@@ -190,10 +278,11 @@
     <parent link="chassis_link" />
     <child link="imu_link" />
+    <origin xyz="${imu_offset_x} ${imu_offset_y} ${imu_offset_z}" rpy="0 0 0"/>
   </joint>
   <link name="mid_mount" />
   <joint name="mid_mount_joint" type="fixed">
-    <parent link="base_link" />
+    <parent link="riser_link" />
     <child link="mid_mount" />
-    <origin xyz="0 0 ${deck_height}" rpy="0 0 0"/>
+    <origin xyz="0 0 ${riser_height + deck_thickness}" rpy="0 0 0"/>
   </joint>
   <!-- Bring in simulation data for Gazebo. -->
